Commit message: Modify URDF converter to use collision geometry instead of visual
Co-authored-by: 20niship <81469647+20niship@users.noreply.github.com>

File: tests/robot_with_collision.urdf (robot description, URDF)
Before this commit: robot robot_with_mesh, 3 links, 2 joints
Links:
- added link link3, mass 0.3; collision box size=0.15 0.15 0.15; visual box size=0.15 0.15 0.15
- link base_link: geometry collision box size=0.2 0.2 0.2; visual mesh filename=package://robot_description/meshes/base.stl scale=1.0 1.0 1.0
- link link1: geometry collision cylinder length=0.4 radius=0.05; visual mesh filename=meshes/link1.obj scale=0.5 0.5 0.5
- link link2: geometry collision sphere radius=0.1; visual mesh filename=meshes/link2.obj
Joints:
- added joint joint3: type revolute, parent link2, child link3, origin xyz=0 0 0.2 rpy=0 0 0, axis 1 0 0, limit lower=-1.57 upper=1.57 effort=3.0 velocity=1.0
